File: KiCad/picow_plant_moisture_sensor/picow_plant_moisture_sensor.kicad_pcb (KiCad board)
At the start: 4 copper layers, 94.6 x 64.1 mm, 59 parts, among them J1 Conn_01x03, J10 Conn_01x03, J11 Conn_01x03, J12 Conn_01x03, J13 Conn_02x03_Odd_Even, J14 Conn_01x03, J15 Conn_01x03, J16 Conn_01x03, J17 Conn_01x03, J2 Conn_01x03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

Commit message: Rev1 ordered
Parts:
- D1, D2, D3: footprint LED_SMD:LED_0402_1005Metric -> LED_SMD:LED_0603_1608Metric
- SW1, SW2, SW3, SW4: footprint Button_Switch_SMD:SW_Push_1P1T_NO_Vertical_Wuerth_434133025816 -> Button_Switch_THT:SW_PUSH_6mm
- moved R15 38.8 mm to (116.6, 49.0)
- moved SW2 15.9 mm to (86.2, 50.0)
- moved R14 14.4 mm to (115.2, 57.2)
- moved R13 10.8 mm to (114.7, 62.3)
- moved SW3 7.08 mm to (99.5, 50.0)
- moved R20 5.79 mm to (147.1, 73.1), turned to 180 degrees
- moved R19 5.38 mm to (147.1, 69.3), turned to 180 degrees
- moved R18 5.20 mm to (147.1, 65.5), turned to 180 degrees
- moved SW4 3.92 mm to (112.8, 50.0)
- moved D1 3.70 mm to (152.1, 62.9), turned to 180 degrees
- moved D2 2.94 mm to (152.1, 66.8), turned to 180 degrees
- moved D3 2.69 mm to (152.1, 70.6), turned to 180 degrees
- moved C1 0.16 mm to (105.0, 63.6)
Connections:
- R13 pad 1: /GPIO0 -> /GPIO4
- R14 pad 1: /GPIO6 -> /GPIO2
- R15 pad 1: /GPIO11 -> /GPIO0
- R18 pad 2: /GPIO2 -> /GPIO28
- R19 pad 2: /GPIO3 -> /GPIO27
- R20 pad 2: /GPIO4 -> /GPIO26
Routing:
- net /GPIO3: track 58.0 -> 0.00 mm
- net /GPIO4: track 61.5 -> 6.95 mm
- net /GPIO2: track 58.1 -> 6.67 mm
- net Net-(R15-Pad2): track 44.9 -> 11.4 mm, vias 2 -> 0
- net Net-(R13-Pad2): track 16.8 -> 41.5 mm
- net +3V3: track 27.1 -> 16.8 mm, vias 14 -> 8
- net /GPIO27: track 0.00 -> 7.95 mm
- net /GPIO26: track 0.00 -> 7.42 mm
- net /GPIO28: track 0.00 -> 7.42 mm
- net GND: track 25.3 -> 32.3 mm
- net /GPIO11: track 6.83 -> 0.00 mm
- net /GPIO6: track 5.85 -> 0.00 mm
- net /RUN: track 13.0 -> 17.0 mm
- net /GPIO9: track 53.4 -> 50.1 mm
- net Net-(D2-A): track 1.82 -> 4.83 mm
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Other:
- board text added: "- Ain - +3V3 - GND"
- board text removed: "UART"
