File: KiCad/picow_plant_moisture_sensor/picow_plant_moisture_sensor.kicad_sch (KiCad schematic)
At the start: 59 parts, among them J1 Conn_01x03, J10 Conn_01x03, J11 Conn_01x03, J12 Conn_01x03, J13 Conn_02x03_Odd_Even, J14 Conn_01x03, J15 Conn_01x03, J16 Conn_01x03, J17 Conn_01x03, J2 Conn_01x03, J3 Conn_01x03, J4 Conn_01x03, J5 Conn_01x03, J6 Conn_01x03, J7 Conn_01x03, J8 Conn_01x03, J9 Conn_01x03, SW1 SW_Push, SW2 SW_Push, SW3 SW_Push, SW4 SW_Push, U1 ADS1115IDGS, U2 PicoW, U3 ADS1115IDGS, U4 ADS1115IDGS, U5 ADS1115IDGS

Commit message: Complete PCB design with component references
Parts:
- C1, C2, C3, C4: LCSC (none) -> C1525
- D1, D2, D3: LCSC (none) -> C88330
- R1, R2: LCSC (none) -> C351692
- R10, R11, R12, R16, R17, R3, R4, R5, R6, R7, R8, R9: LCSC (none) -> C15402
- R13, R14, R15: LCSC (none) -> C844716
- R18, R19, R20: LCSC (none) -> C100375
- U1, U3, U4, U5: LCSC (none) -> C37593
Changed lines of the file:
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@@
+      (effects (font (size 1.27 1.27)) hide)
+    )
+    (property "LCSC" "C844716" (at 284.48 41.91 0)
       (effects (font (size 1.27 1.27)) hide)
     )
@@
       (effects (font (size 1.27 1.27)) hide)
     )
+    (property "LCSC" "C844716" (at 284.48 78.74 0)
+      (effects (font (size 1.27 1.27)) hide)
+    )
     (pin "1")
     (pin "2")
@@
     )
     (property "Datasheet" "~" (at 281.94 119.38 0)
+      (effects (font (size 1.27 1.27)) hide)
+    )
+    (property "LCSC" "C844716" (at 284.48 115.57 0)
       (effects (font (size 1.27 1.27)) hide)
     )
@@
       (effects (font (size 1.27 1.27)) hide)
     )
+    (property "LCSC" "C1525" (at 44.831 179.1716 0)
+      (effects (font (size 1.27 1.27)) hide)
+    )
     (pin "1")
     (pin "2")
@@
       (effects (font (size 1.27 1.27)) hide)
     )
+    (property "LCSC" "C15402" (at 224.79 200.66 0)
+      (effects (font (size 1.27 1.27)) hide)
+    )
     (pin "1")
     (pin "2")
@@
     )
     (property "Datasheet" "~" (at 25.4 110.49 0)
+      (effects (font (size 1.27 1.27)) hide)
+    )
+    (property "LCSC" "C351692" (at 27.94 106.68 0)
       (effects (font (size 1.27 1.27)) hide)
     )
@@
       (effects (font (size 1.27 1.27)) hide)
     )
+    (property "LCSC" "C15402" (at 283.21 166.37 0)
+      (effects (font (size 1.27 1.27)) hide)
+    )
     (pin "1")
     (pin "2")
@@
       (effects (font (size 1.27 1.27)) hide)
     )
+    (property "LCSC" "C15402" (at 130.81 166.37 0)
+      (effects (font (size 1.27 1.27)) hide)
+    )
     (pin "1")
     (pin "2")
@@
       (effects (font (size 1.27 1.27)) hide)
     )
+    (property "LCSC" "C15402" (at 78.74 200.66 0)
+      (effects (font (size 1.27 1.27)) hide)
+    )
     (pin "1")
     (pin "2")
@@
     )
     (property "Datasheet" "~" (at 55.88 170.18 0)
+      (effects (font (size 1.27 1.27)) hide)
+    )
+    (property "LCSC" "C15402" (at 58.42 166.37 0)
       (effects (font (size 1.27 1.27)) hide)
     )
@@
     )
     (property "Datasheet" "http://www.ti.com/lit/ds/symlink/ads1113.pdf" (at 54.61 222.25 0)
+      (effects (font (size 1.27 1.27)) hide)
+    )
+    (property "LCSC" "C37593" (at 58.0741 184.15 0)
       (effects (font (size 1.27 1.27)) hide)
     )
@@
       (effects (font (size 1.27 1.27)) hide)
     )
+    (property "LCSC" "C15402" (at 303.53 200.66 0)
+      (effects (font (size 1.27 1.27)) hide)
+    )
     (pin "1")
     (pin "2")
@@
       (effects (font (size 1.27 1.27)) hide)
     )
+    (property "LCSC" "C15402" (at 303.53 207.01 0)
+      (effects (font (size 1.27 1.27)) hide)
+    )
     (pin "1")
     (pin "2")
@@
       (effects (font (size 1.27 1.27)) hide)
     )
+    (property "LCSC" "C100375" (at 181.61 83.82 0)
+      (effects (font (size 1.27 1.27)) hide)
+    )
     (pin "1")
     (pin "2")
@@
       (effects (font (size 1.27 1.27)) hide)
     )
+    (property "LCSC" "C100375" (at 181.61 72.39 0)
+      (effects (font (size 1.27 1.27)) hide)
+    )
     (pin "1")
     (pin "2")
@@
     )
     (property "Datasheet" "~" (at 147.32 198.12 0)
+      (effects (font (size 1.27 1.27)) hide)
+    )
+    (property "LCSC" "C15402" (at 151.13 200.66 0)
       (effects (font (size 1.27 1.27)) hide)
     )
@@
     )
     (property "Datasheet" "http://www.ti.com/lit/ds/symlink/ads1113.pdf" (at 127 222.25 0)
+      (effects (font (size 1.27 1.27)) hide)
+    )
+    (property "LCSC" "C37593" (at 128.27 199.39 0)
       (effects (font (size 1.27 1.27)) hide)
     )
@@
       (effects (font (size 1.27 1.27)) hide)
     )
+    (property "LCSC" "C15402" (at 78.74 207.01 0)
+      (effects (font (size 1.27 1.27)) hide)
+    )
     (pin "1")
     (pin "2")
@@
       (effects (font (size 1.27 1.27)) hide)
     )
+    (property "LCSC" "C1525" (at 117.221 179.1716 0)
+      (effects (font (size 1.27 1.27)) hide)
+    )
     (pin "1")
     (pin "2")
@@
     )
     (property "Datasheet" "~" (at 201.93 170.18 0)
+      (effects (font (size 1.27 1.27)) hide)
+    )
+    (property "LCSC" "C15402" (at 204.47 166.37 0)
       (effects (font (size 1.27 1.27)) hide)
     )
@@
       (effects (font (size 1.27 1.27)) hide)
     )
+    (property "LCSC" "C88330" (at 160.9725 74.93 0)
+      (effects (font (size 1.27 1.27)) hide)
+    )
     (pin "2")
     (pin "1")
@@
       (effects (font (size 1.27 1.27)) hide)
     )
+    (property "LCSC" "C1525" (at 190.881 179.1716 0)
+      (effects (font (size 1.27 1.27)) hide)
+    )
     (pin "1")
     (pin "2")
@@
       (effects (font (size 1.27 1.27)) hide)
     )
+    (property "LCSC" "C1525" (at 269.621 179.1716 0)
+      (effects (font (size 1.27 1.27)) hide)
+    )
     (pin "1")
     (pin "2")
@@
       (effects (font (size 1.27 1.27)) hide)
     )
+    (property "LCSC" "C15402" (at 151.13 207.01 0)
+      (effects (font (size 1.27 1.27)) hide)
+    )
     (pin "1")
     (pin "2")
@@
     )
     (property "Datasheet" "~" (at 220.98 204.47 0)
+      (effects (font (size 1.27 1.27)) hide)
+    )
+    (property "LCSC" "C15402" (at 224.79 207.01 0)
       (effects (font (size 1.27 1.27)) hide)
     )
@@
     )
     (property "Datasheet" "http://www.ti.com/lit/ds/symlink/ads1113.pdf" (at 200.66 222.25 0)
+      (effects (font (size 1.27 1.27)) hide)
+    )
+    (property "LCSC" "C37593" (at 204.1241 184.15 0)
       (effects (font (size 1.27 1.27)) hide)
     )
@@
       (effects (font (size 1.27 1.27)) hide)
     )
+    (property "LCSC" "C88330" (at 160.9725 52.07 0)
+      (effects (font (size 1.27 1.27)) hide)
+    )
     (pin "2")
     (pin "1")
@@
     )
     (property "Datasheet" "~" (at 16.51 110.49 0)
+      (effects (font (size 1.27 1.27)) hide)
+    )
+    (property "LCSC" "C351692" (at 19.05 106.68 0)
       (effects (font (size 1.27 1.27)) hide)
     )
@@
       (effects (font (size 1.27 1.27)) hide)
     )
+    (property "LCSC" "C88330" (at 160.9725 63.5 0)
+      (effects (font (size 1.27 1.27)) hide)
+    )
     (pin "2")
     (pin "1")
@@
     )
     (property "Datasheet" "~" (at 177.8 58.42 0)
+      (effects (font (size 1.27 1.27)) hide)
+    )
+    (property "LCSC" "C100375" (at 181.61 60.96 0)
       (effects (font (size 1.27 1.27)) hide)
     )
@@
       (effects (font (size 1.27 1.27)) hide)
     )
+    (property "LCSC" "C37593" (at 282.8641 184.15 0)
+      (effects (font (size 1.27 1.27)) hide)
+    )

Commit message: Rev1 ordered
Parts:
- D1, D2, D3: footprint LED_SMD:LED_0402_1005Metric -> LED_SMD:LED_0603_1608Metric; LCSC C88330 -> C2290
- R1, R2: LCSC C351692 -> C25900
- R10, R11, R12, R16, R17, R3, R4, R5, R6, R7, R8, R9: LCSC C15402 -> C21189
- R13, R14, R15: LCSC C844716 -> C11702
- R18, R19, R20: LCSC C100375 -> C25104
- SW1, SW2, SW3, SW4: footprint Button_Switch_SMD:SW_Push_1P1T_NO_Vertical_Wuerth_434133025816 -> Button_Switch_THT:SW_PUSH_6mm
Connections:
- net GPIO0: now also R15.1; no longer R13.1
- net GPIO11: no longer R15.1
- net GPIO2: now also R14.1; no longer R18.2
- net GPIO26: now also R20.2
- net GPIO27: now also R19.2
- net GPIO28: now also R18.2
- net GPIO3: no longer R19.2
- net GPIO4: now also R13.1; no longer R20.2
- net GPIO6: no longer R14.1
Changed lines of the file:
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@@
     (effects (font (size 1.27 1.27)) (justify right bottom))
   )
-  (label "GPIO4" (at 187.96 81.28 0) (fields_autoplaced)
+  (label "GPIO26" (at 187.96 81.28 0) (fields_autoplaced)
     (effects (font (size 1.27 1.27)) (justify left bottom))
   )
@@
     (effects (font (size 1.27 1.27)) (justify right bottom))
   )
-  (label "GPIO3" (at 187.96 69.85 0) (fields_autoplaced)
+  (label "GPIO27" (at 187.96 69.85 0) (fields_autoplaced)
     (effects (font (size 1.27 1.27)) (justify left bottom))
   )
@@
     (effects (font (size 1.27 1.27)) (justify left bottom))
   )
-  (label "GPIO6" (at 297.18 88.9 0) (fields_autoplaced)
+  (label "GPIO2" (at 297.18 88.9 0) (fields_autoplaced)
     (effects (font (size 1.27 1.27)) (justify left bottom))
   )
@@
     (effects (font (size 1.27 1.27)) (justify left bottom))
   )
-  (label "GPIO2" (at 187.96 58.42 0) (fields_autoplaced)
+  (label "GPIO28" (at 187.96 58.42 0) (fields_autoplaced)
     (effects (font (size 1.27 1.27)) (justify left bottom))
   )
@@
     (effects (font (size 1.27 1.27)) (justify left bottom))
   )
-  (label "GPIO11" (at 297.18 125.73 0) (fields_autoplaced)
+  (label "GPIO0" (at 297.18 125.73 0) (fields_autoplaced)
     (effects (font (size 1.27 1.27)) (justify left bottom))
   )
@@
     (effects (font (size 1.27 1.27)) (justify left bottom))
   )
-  (label "GPIO0" (at 297.18 52.07 0) (fields_autoplaced)
+  (label "GPIO4" (at 297.18 52.07 0) (fields_autoplaced)
     (effects (font (size 1.27 1.27)) (justify left bottom))
   )
@@
       (effects (font (size 1.27 1.27)) (justify left))
     )
-    (property "Footprint" "Button_Switch_SMD:SW_Push_1P1T_NO_Vertical_Wuerth_434133025816" (at 287.02 35.56 0)
+    (property "Footprint" "Button_Switch_THT:SW_PUSH_6mm" (at 287.02 35.56 0)
       (effects (font (size 1.27 1.27)) hide)
     )
@@
       (effects (font (size 1.27 1.27)) hide)
     )
-    (property "LCSC" "C844716" (at 284.48 41.91 0)
+    (property "LCSC" "C11702" (at 284.48 41.91 0)
       (effects (font (size 1.27 1.27)) hide)
     )
@@
       (effects (font (size 1.27 1.27)) (justify left))
     )
-    (property "Footprint" "Button_Switch_SMD:SW_Push_1P1T_NO_Vertical_Wuerth_434133025816" (at 287.02 72.39 0)
+    (property "Footprint" "Button_Switch_THT:SW_PUSH_6mm" (at 287.02 72.39 0)
       (effects (font (size 1.27 1.27)) hide)
     )
@@
       (effects (font (size 1.27 1.27)) hide)
     )
-    (property "LCSC" "C844716" (at 284.48 78.74 0)
+    (property "LCSC" "C11702" (at 284.48 78.74 0)
       (effects (font (size 1.27 1.27)) hide)
     )
@@
       (effects (font (size 1.27 1.27)) (justify left))
     )
-    (property "Footprint" "Button_Switch_SMD:SW_Push_1P1T_NO_Vertical_Wuerth_434133025816" (at 287.02 109.22 0)
+    (property "Footprint" "Button_Switch_THT:SW_PUSH_6mm" (at 287.02 109.22 0)
       (effects (font (size 1.27 1.27)) hide)
     )
@@
       (effects (font (size 1.27 1.27)) hide)
     )
-    (property "LCSC" "C844716" (at 284.48 115.57 0)
+    (property "LCSC" "C11702" (at 284.48 115.57 0)
       (effects (font (size 1.27 1.27)) hide)
     )
@@
       (effects (font (size 1.27 1.27)) (justify left))
     )
-    (property "Footprint" "Button_Switch_SMD:SW_Push_1P1T_NO_Vertical_Wuerth_434133025816" (at 127 110.49 0)
+    (property "Footprint" "Button_Switch_THT:SW_PUSH_6mm" (at 127 110.49 0)
       (effects (font (size 1.27 1.27)) hide)
     )
@@
       (effects (font (size 1.27 1.27)) hide)
     )
-    (property "LCSC" "C15402" (at 224.79 200.66 0)
+    (property "LCSC" "C21189" (at 224.79 200.66 0)
       (effects (font (size 1.27 1.27)) hide)
     )
@@
       (effects (font (size 1.27 1.27)) hide)
     )
-    (property "LCSC" "C351692" (at 27.94 106.68 0)
+    (property "LCSC" "C25900" (at 27.94 106.68 0)
       (effects (font (size 1.27 1.27)) hide)
     )
@@
       (effects (font (size 1.27 1.27)) hide)
     )
-    (property "LCSC" "C15402" (at 283.21 166.37 0)
+    (property "LCSC" "C21189" (at 283.21 166.37 0)
       (effects (font (size 1.27 1.27)) hide)
     )
@@
       (effects (font (size 1.27 1.27)) hide)
     )
-    (property "LCSC" "C15402" (at 130.81 166.37 0)
+    (property "LCSC" "C21189" (at 130.81 166.37 0)
       (effects (font (size 1.27 1.27)) hide)
     )
@@
       (effects (font (size 1.27 1.27)) hide)
     )
-    (property "LCSC" "C15402" (at 78.74 200.66 0)
+    (property "LCSC" "C21189" (at 78.74 200.66 0)
       (effects (font (size 1.27 1.27)) hide)
     )
@@
       (effects (font (size 1.27 1.27)) hide)
     )
-    (property "LCSC" "C15402" (at 58.42 166.37 0)
+    (property "LCSC" "C21189" (at 58.42 166.37 0)
       (effects (font (size 1.27 1.27)) hide)
     )
@@
       (effects (font (size 1.27 1.27)) hide)
     )
-    (property "LCSC" "C15402" (at 303.53 200.66 0)
+    (property "LCSC" "C21189" (at 303.53 200.66 0)
       (effects (font (size 1.27 1.27)) hide)
     )
@@
       (effects (font (size 1.27 1.27)) hide)
     )
-    (property "LCSC" "C15402" (at 303.53 207.01 0)
+    (property "LCSC" "C21189" (at 303.53 207.01 0)
       (effects (font (size 1.27 1.27)) hide)
     )
@@
       (effects (font (size 1.27 1.27)) hide)
     )
-    (property "LCSC" "C100375" (at 181.61 83.82 0)
+    (property "LCSC" "C25104" (at 181.61 83.82 0)
       (effects (font (size 1.27 1.27)) hide)
     )
@@
       (effects (font (size 1.27 1.27)) hide)
     )
-    (property "LCSC" "C100375" (at 181.61 72.39 0)
+    (property "LCSC" "C25104" (at 181.61 72.39 0)
       (effects (font (size 1.27 1.27)) hide)
     )
@@
       (effects (font (size 1.27 1.27)) hide)
     )
-    (property "LCSC" "C15402" (at 151.13 200.66 0)
+    (property "LCSC" "C21189" (at 151.13 200.66 0)
       (effects (font (size 1.27 1.27)) hide)
     )
@@
       (effects (font (size 1.27 1.27)) hide)
     )
-    (property "LCSC" "C15402" (at 78.74 207.01 0)
+    (property "LCSC" "C21189" (at 78.74 207.01 0)
       (effects (font (size 1.27 1.27)) hide)
     )
@@
       (effects (font (size 1.27 1.27)) hide)
     )
-    (property "LCSC" "C15402" (at 204.47 166.37 0)
+    (property "LCSC" "C21189" (at 204.47 166.37 0)
       (effects (font (size 1.27 1.27)) hide)
     )
@@
       (effects (font (size 1.27 1.27)))
     )
-    (property "Footprint" "LED_SMD:LED_0402_1005Metric" (at 162.56 81.28 0)
+    (property "Footprint" "LED_SMD:LED_0603_1608Metric" (at 162.56 81.28 0)
       (effects (font (size 1.27 1.27)) hide)
     )
@@
       (effects (font (size 1.27 1.27)) hide)
     )
-    (property "LCSC" "C88330" (at 160.9725 74.93 0)
+    (property "LCSC" "C2290" (at 160.9725 74.93 0)
       (effects (font (size 1.27 1.27)) hide)
     )
@@
       (effects (font (size 1.27 1.27)) hide)
     )
-    (property "LCSC" "C15402" (at 151.13 207.01 0)
+    (property "LCSC" "C21189" (at 151.13 207.01 0)
       (effects (font (size 1.27 1.27)) hide)
     )
@@
       (effects (font (size 1.27 1.27)) hide)
     )
-    (property "LCSC" "C15402" (at 224.79 207.01 0)
+    (property "LCSC" "C21189" (at 224.79 207.01 0)
       (effects (font (size 1.27 1.27)) hide)
     )
@@
       (effects (font (size 1.27 1.27)))
     )
-    (property "Footprint" "LED_SMD:LED_0402_1005Metric" (at 162.56 58.42 0)
+    (property "Footprint" "LED_SMD:LED_0603_1608Metric" (at 162.56 58.42 0)
       (effects (font (size 1.27 1.27)) hide)
     )
@@
       (effects (font (size 1.27 1.27)) hide)
     )
-    (property "LCSC" "C88330" (at 160.9725 52.07 0)
+    (property "LCSC" "C2290" (at 160.9725 52.07 0)
       (effects (font (size 1.27 1.27)) hide)
     )
@@
       (effects (font (size 1.27 1.27)) hide)
     )
-    (property "LCSC" "C351692" (at 19.05 106.68 0)
+    (property "LCSC" "C25900" (at 19.05 106.68 0)
       (effects (font (size 1.27 1.27)) hide)
     )
@@
       (effects (font (size 1.27 1.27)))
     )
-    (property "Footprint" "LED_SMD:LED_0402_1005Metric" (at 162.56 69.85 0)
+    (property "Footprint" "LED_SMD:LED_0603_1608Metric" (at 162.56 69.85 0)
       (effects (font (size 1.27 1.27)) hide)
     )
@@
       (effects (font (size 1.27 1.27)) hide)
     )
-    (property "LCSC" "C88330" (at 160.9725 63.5 0)
+    (property "LCSC" "C2290" (at 160.9725 63.5 0)
       (effects (font (size 1.27 1.27)) hide)
     )
@@
       (effects (font (size 1.27 1.27)) hide)
     )
-    (property "LCSC" "C100375" (at 181.61 60.96 0)
+    (property "LCSC" "C25104" (at 181.61 60.96 0)
       (effects (font (size 1.27 1.27)) hide)
     )

Commit message: Add rev2 (#33)
Parts:
- added R21, R22: 5k, Resistor_SMD:R_0603_1608Metric, symbol Device:R
- added TP3, TP4: TestPoint, TestPoint:TestPoint_Pad_D2.0mm, symbol Connector:TestPoint
- added U6: 24LC16, 24LC16B-I_SN:SOIC127P600X175-8N, symbol Memory_EEPROM:24LC16
- C1, C2, C3, C4: footprint Capacitor_SMD:C_0402_1005Metric -> Capacitor_SMD:C_0603_1608Metric
- R1, R13, R14, R15, R18, R19, R2, R20: footprint Resistor_SMD:R_0402_1005Metric -> Resistor_SMD:R_0603_1608Metric
Connections:
- net +3V3: now also R21.2, R22.2, U6.8 (VCC)
- net AIN0: now also U1.4 (AIN0); no longer U1.7 (AIN3)
- net AIN1: now also U1.5 (AIN1); no longer U1.6 (AIN2)
- net AIN10: now also U4.6 (AIN2); no longer U4.5 (AIN1)
- net AIN11: now also U4.7 (AIN3); no longer U4.4 (AIN0)
- net AIN12: now also U5.4 (AIN0); no longer U5.7 (AIN3)
- net AIN13: now also U5.5 (AIN1); no longer U5.6 (AIN2)
- net AIN14: now also U5.6 (AIN2); no longer U5.5 (AIN1)
- net AIN15: now also U5.7 (AIN3); no longer U5.4 (AIN0)
- net AIN2: now also U1.6 (AIN2); no longer U1.5 (AIN1)
- net AIN3: now also U1.7 (AIN3); no longer U1.4 (AIN0)
- net AIN4: now also U3.4 (AIN0); no longer U3.7 (AIN3)
- net AIN5: now also U3.5 (AIN1); no longer U3.6 (AIN2)
- net AIN6: now also U3.6 (AIN2); no longer U3.5 (AIN1)
- net AIN7: now also U3.7 (AIN3); no longer U3.4 (AIN0)
- net AIN8: now also U4.4 (AIN0); no longer U4.7 (AIN3)
- net AIN9: now also U4.5 (AIN1); no longer U4.6 (AIN2)
- net GND: now also J13.4 (Pin_4), J13.5 (Pin_5), U6.4 (GND), U6.7 (WP)
- net GPIO16: now also J13.3 (Pin_3)
- net GPIO17: now also J13.1 (Pin_1)
- net GPIO20: now also R22.1, U6.5 (SDA); no longer J13.3 (Pin_3), J13.4 (Pin_4)
- net GPIO21: now also R21.1, U6.6 (SCL); no longer J13.1 (Pin_1), J13.2 (Pin_2)
- net GPIO8: now also R11.2, R17.2, R5.2, R8.2; no longer R10.2, R16.2, R4.2, R7.2
- net GPIO9: now also R10.2, R16.2, R4.2, R7.2; no longer R11.2, R17.2, R5.2, R8.2
- net SWCLK: now also J13.2 (Pin_2); no longer J13.6 (Pin_6)
- net SWDIO: now also J13.6 (Pin_6); no longer J13.5 (Pin_5)
- new net SCL: TP3.1
- new net SDA: TP4.1
- no-connect marks 25 -> 26
Other:
- note added: "UART0_RX"
- note added: "UART0_TX"
- note removed: "UART1_RX"
- note removed: "UART1_TX"
- moved on the sheet: SW1
