File: KiCad/picow_plant_moisture_sensor/picow_plant_moisture_sensor.kicad_sch (KiCad schematic)
At the start: 64 parts, among them J1 Conn_01x03, J10 Conn_01x03, J11 Conn_01x03, J12 Conn_01x03, J13 Conn_02x03_Odd_Even, J14 Conn_01x03, J15 Conn_01x03, J16 Conn_01x03, J17 Conn_01x03, J2 Conn_01x03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

Commit message: 32 board bring up (#35)
* Add rev2

* Add eeprom cap and I2C test points
Parts:
- added C5: 100n, Capacitor_SMD:C_0603_1608Metric, symbol Device:C
- added TP5, TP6: TestPoint, TestPoint:TestPoint_Pad_D2.0mm, symbol Connector:TestPoint
Connections:
- net SCL is gone; now on net GPIO9: TP3.1
- net SDA is gone; now on net GPIO8: TP4.1
- net +3V3: now also C5.1
- net GND: now also J13.3 (Pin_3), C5.2; no longer J13.5 (Pin_5)
- net GPIO16: now also J13.5 (Pin_5); no longer J13.3 (Pin_3)
- net GPIO20: now also TP5.1
- net GPIO21: now also TP6.1
Changed lines of the file:
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@@
   (junction (at 53.34 107.95) (diameter 0) (color 0 0 0 0)
   )
+  (junction (at 144.78 129.54) (diameter 0) (color 0 0 0 0)
+  )
   (no_connect (at 107.95 105.41))
   (no_connect (at 39.37 105.41))
@@
     (stroke (width 0) (type default))
   )
+  (wire (pts (xy 208.28 123.19) (xy 205.74 123.19))
+    (stroke (width 0) (type default))
+  )
   (wire (pts (xy 181.61 69.85) (xy 194.31 69.85))
     (stroke (width 0) (type default))
@@
     (stroke (width 0) (type default))
   )
-  (wire (pts (xy 198.12 128.27) (xy 198.12 127))
-    (stroke (width 0) (type default))
-  )
   (wire (pts (xy 196.85 255.27) (xy 196.85 251.46))
     (stroke (width 0) (type default))
@@
     (stroke (width 0) (type default))
   )
+  (wire (pts (xy 209.55 124.46) (xy 208.28 124.46))
+    (stroke (width 0) (type default))
+  )
   (wire (pts (xy 20.32 100.33) (xy 20.32 101.6))
     (stroke (width 0) (type default))
@@
     (stroke (width 0) (type default))
   )
-  (wire (pts (xy 198.12 127) (xy 209.55 127))
-    (stroke (width 0) (type default))
-  )
   (wire (pts (xy 50.8 254) (xy 50.8 250.19))
     (stroke (width 0) (type default))
@@
     (stroke (width 0) (type default))
   )
+  (wire (pts (xy 208.28 124.46) (xy 208.28 123.19))
+    (stroke (width 0) (type default))
+  )
   (wire (pts (xy 173.99 69.85) (xy 166.37 69.85))
     (stroke (width 0) (type default))
@@
     (stroke (width 0) (type default))
   )
+  (wire (pts (xy 53.34 26.67) (xy 53.34 33.02))
+    (stroke (width 0) (type default))
+  )
   (wire (pts (xy 123.19 255.27) (xy 123.19 251.46))
     (stroke (width 0) (type default))
@@
     (stroke (width 0) (type default))
   )
-  (wire (pts (xy 144.78 128.27) (xy 144.78 133.35))
+  (wire (pts (xy 144.78 128.27) (xy 144.78 129.54))
     (stroke (width 0) (type default))
   )
@@
     (stroke (width 0) (type default))
   )
+  (wire (pts (xy 127 129.54) (xy 144.78 129.54))
+    (stroke (width 0) (type default))
+  )
   (wire (pts (xy 290.83 204.47) (xy 294.64 204.47))
     (stroke (width 0) (type default))
@@
     (stroke (width 0) (type default))
   )
-  (wire (pts (xy 36.83 273.05) (xy 50.8 273.05))
+  (wire (pts (xy 195.58 127) (xy 209.55 127))
     (stroke (width 0) (type default))
   )
-  (wire (pts (xy 181.61 274.32) (xy 196.85 274.32))
+  (wire (pts (xy 36.83 273.05) (xy 50.8 273.05))
     (stroke (width 0) (type default))
   )
-  (wire (pts (xy 209.55 124.46) (xy 195.58 124.46))
+  (wire (pts (xy 181.61 274.32) (xy 196.85 274.32))
     (stroke (width 0) (type default))
   )
@@
     (stroke (width 0) (type default))
   )
+  (wire (pts (xy 67.31 26.67) (xy 67.31 33.02))
+    (stroke (width 0) (type default))
+  )
   (wire (pts (xy 212.09 201.93) (xy 215.9 201.93))
     (stroke (width 0) (type default))
   )
+  (wire (pts (xy 127 130.81) (xy 127 129.54))
+    (stroke (width 0) (type default))
+  )
   (wire (pts (xy 129.54 107.95) (xy 129.54 109.22))
     (stroke (width 0) (type default))
@@
     (stroke (width 0) (type default))
   )
+  (wire (pts (xy 144.78 129.54) (xy 144.78 133.35))
+    (stroke (width 0) (type default))
+  )
   (wire (pts (xy 36.83 223.52) (xy 50.8 223.52))
     (stroke (width 0) (type default))
@@
     (effects (font (size 1.27 1.27)) (justify left bottom))
   )
-  (text "UART0_TX " (at 184.15 124.46 0)
+  (text "UART0_TX " (at 184.15 127 0)
     (effects (font (size 1.27 1.27)) (justify left bottom))
   )
@@
     (effects (font (size 1.27 1.27)) (justify left bottom))
   )
-  (label "SCL" (at 99.06 26.67 0) (fields_autoplaced)
+  (label "SCL1" (at 99.06 26.67 0) (fields_autoplaced)
     (effects (font (size 1.27 1.27)) (justify left bottom))
   )
@@
     (effects (font (size 1.27 1.27)) (justify right bottom))
   )
-  (label "SDA" (at 85.09 26.67 0) (fields_autoplaced)
+  (label "SDA1" (at 85.09 26.67 0) (fields_autoplaced)
     (effects (font (size 1.27 1.27)) (justify left bottom))
   )
@@
     (effects (font (size 1.27 1.27)) (justify left bottom))
   )
-  (label "GPIO16" (at 195.58 124.46 0) (fields_autoplaced)
+  (label "GPIO16" (at 195.58 127 0) (fields_autoplaced)
     (effects (font (size 1.27 1.27)) (justify left bottom))
   )
@@
     (effects (font (size 1.27 1.27)) (justify left bottom))
   )
+  (label "SCL0" (at 67.31 26.67 0) (fields_autoplaced)
+    (effects (font (size 1.27 1.27)) (justify left bottom))
+  )
   (label "SDA1" (at 83.82 204.47 0) (fields_autoplaced)
     (effects (font (size 1.27 1.27)) (justify left bottom))
@@
     (effects (font (size 1.27 1.27)) (justify left bottom))
   )
+  (label "SDA0" (at 53.34 26.67 0) (fields_autoplaced)
+    (effects (font (size 1.27 1.27)) (justify left bottom))
+  )
   (symbol (lib_id "RPi_Pico:PicoW") (at 73.66 114.3 0) (unit 1)
     (in_bom yes) (on_board yes) (dnp no)
@@
     )
   )
+  (symbol (lib_id "Device:C") (at 127 134.62 0) (unit 1)
+    (in_bom yes) (on_board yes) (dnp no)
+    (property "Reference" "C5" (at 129.921 133.4516 0)
+      (effects (font (size 1.27 1.27)) (justify left))
+    )
+    (property "Value" "100n" (at 129.921 135.763 0)
+      (effects (font (size 1.27 1.27)) (justify left))
+    )
+    (property "Footprint" "Capacitor_SMD:C_0603_1608Metric" (at 127.9652 138.43 0)
+      (effects (font (size 1.27 1.27)) hide)
+    )
+    (property "Datasheet" "~" (at 127 134.62 0)
+      (effects (font (size 1.27 1.27)) hide)
+    )
+    (property "LCSC" "C1525" (at 129.921 133.4516 0)
+      (effects (font (size 1.27 1.27)) hide)
+    )
+    (pin "1")
+    (pin "2")
+    (instances
+      (project "picow_plant_moisture_sensor"
+        (path "/7e7c068a-a341-4358-ab45-53bb7a793d6f"
+          (reference "C5") (unit 1)
+        )
+      )
+    )
+  )
   (symbol (lib_id "Device:R") (at 74.93 198.12 90) (unit 1)
     (in_bom yes) (on_board yes) (dnp no)
@@
     )
   )
+  (symbol (lib_id "Connector:TestPoint") (at 67.31 33.02 180) (unit 1)
+    (in_bom yes) (on_board yes) (dnp no) (fields_autoplaced)
+    (property "Reference" "TP6" (at 69.85 35.052 0)
+      (effects (font (size 1.27 1.27)) (justify right))
+    )
+    (property "Value" "TestPoint" (at 69.85 37.592 0)
+      (effects (font (size 1.27 1.27)) (justify right))
+    )
+    (property "Footprint" "TestPoint:TestPoint_Pad_D2.0mm" (at 62.23 33.02 0)
+      (effects (font (size 1.27 1.27)) hide)
+    )
+    (property "Datasheet" "~" (at 62.23 33.02 0)
+      (effects (font (size 1.27 1.27)) hide)
+    )
+    (pin "1")
+    (instances
+      (project "picow_plant_moisture_sensor"
+        (path "/7e7c068a-a341-4358-ab45-53bb7a793d6f"
+          (reference "TP6") (unit 1)
+        )
+      )
+    )
+  )
   (symbol (lib_id "power:+3.3V") (at 109.22 224.79 0) (unit 1)
     (in_bom yes) (on_board yes) (dnp no)
@@
     )
   )
-  (symbol (lib_id "power:GND") (at 198.12 128.27 0) (unit 1)
+  (symbol (lib_id "power:GND") (at 205.74 123.19 0) (unit 1)
     (in_bom yes) (on_board yes) (dnp no)
-    (property "Reference" "#PWR063" (at 198.12 134.62 0)
+    (property "Reference" "#PWR063" (at 205.74 129.54 0)
       (effects (font (size 1.27 1.27)) hide)
     )
-    (property "Value" "GND" (at 198.247 132.6642 0)
+    (property "Value" "GND" (at 205.867 127.5842 0)
       (effects (font (size 1.27 1.27)))
     )
-    (property "Footprint" "" (at 198.12 128.27 0)
+    (property "Footprint" "" (at 205.74 123.19 0)
       (effects (font (size 1.27 1.27)) hide)
     )
-    (property "Datasheet" "" (at 198.12 128.27 0)
+    (property "Datasheet" "" (at 205.74 123.19 0)
       (effects (font (size 1.27 1.27)) hide)
     )
@@
     )
   )
+  (symbol (lib_id "Connector:TestPoint") (at 53.34 33.02 180) (unit 1)
+    (in_bom yes) (on_board yes) (dnp no) (fields_autoplaced)
+    (property "Reference" "TP5" (at 55.88 35.052 0)
+      (effects (font (size 1.27 1.27)) (justify right))
+    )
+    (property "Value" "TestPoint" (at 55.88 37.592 0)
+      (effects (font (size 1.27 1.27)) (justify right))
+    )
+    (property "Footprint" "TestPoint:TestPoint_Pad_D2.0mm" (at 48.26 33.02 0)
+      (effects (font (size 1.27 1.27)) hide)
+    )
+    (property "Datasheet" "~" (at 48.26 33.02 0)
+      (effects (font (size 1.27 1.27)) hide)
+    )
+    (pin "1")
+    (instances
+      (project "picow_plant_moisture_sensor"
+        (path "/7e7c068a-a341-4358-ab45-53bb7a793d6f"
+          (reference "TP5") (unit 1)
+        )
+      )
+    )
+  )
   (symbol (lib_id "Analog_ADC:ADS1115IDGS") (at 128.27 199.39 0) (unit 1)
     (in_bom yes) (on_board yes) (dnp no) (fields_autoplaced)
@@
         )
       )
+    )
+  )
+  (symbol (lib_id "power:GND") (at 127 138.43 0) (mirror y) (unit 1)
+    (in_bom yes) (on_board yes) (dnp no)
+    (property "Reference" "#PWR069" (at 127 144.78 0)
+      (effects (font (size 1.27 1.27)) hide)
+    )
+    (property "Value" "GND" (at 126.873 142.8242 0)
+      (effects (font (size 1.27 1.27)))
+    )
+    (property "Footprint" "" (at 127 138.43 0)
+      (effects (font (size 1.27 1.27)) hide)
+    )
+    (property "Datasheet" "" (at 127 138.43 0)
+      (effects (font (size 1.27 1.27)) hide)
+    )
+    (pin "1")
+    (instances
+      (project "picow_plant_moisture_sensor"
+        (path "/7e7c068a-a341-4358-ab45-53bb7a793d6f"
+          (reference "#PWR069") (unit 1)
+        )
+      )

Commit message: Design with RP2040 IC instead of pico board
Parts:
- removed C5: 100n, Capacitor_SMD:C_0603_1608Metric, symbol Device:C
- removed J13: Conn_02x03_Odd_Even, Connector_PinHeader_2.54mm:PinHeader_2x04_P2.54mm_Vertical, symbol Connector_Generic:Conn_02x04_Odd_Even
- removed R21, R22: 5k, Resistor_SMD:R_0603_1608Metric, symbol Device:R
- removed SW1: SW_Push, Button_Switch_THT:SW_PUSH_6mm, symbol Switch:SW_Push
- removed TP5, TP6: TestPoint, TestPoint:TestPoint_Pad_D2.0mm, symbol Connector:TestPoint
- removed U2: PicoW, RaspberryPI PicoW:RPi_PicoW_SMD_TH, symbol RPi_Pico:PicoW
- removed U6: 24LC16, 24LC16B-I_SN:SOIC127P600X175-8N, symbol Memory_EEPROM:24LC16
- added J20: Conn_01x03, Connector_PinHeader_2.54mm:PinHeader_1x03_P2.54mm_Vertical, symbol Connector_Generic:Conn_01x03
- added J21: Conn_01x03, Connector_PinSocket_2.54mm:PinSocket_1x03_P2.54mm_Vertical, symbol Connector_Generic:Conn_01x03
- SW2, SW3, SW4: footprint Button_Switch_THT:SW_PUSH_6mm -> Button_Switch_SMD:SW_SPST_TL3305A
Connections:
- net GND: now also J20.2 (Pin_2), J21.2 (Pin_2)
- net GPIO26 renamed MCU/GPIO26
- net GPIO27 renamed MCU/GPIO27
- net GPIO28 renamed MCU/GPIO28
- net GPIO8 renamed SDA1
- net GPIO9 renamed SCL1
- new net MCU/SWCLK: J21.1 (Pin_1)
- new net MCU/SWD: J21.3 (Pin_3)
- new net MCU/UART0_RX: J20.1 (Pin_1)
- new net MCU/UART0_TX: J20.3 (Pin_3)
- no-connect marks 26 -> 4
Other:
- added sheet MCU (mcu.kicad_sch)
- note added: "Debug"
- note added: "UART"
- note removed: "PicoW"
- note removed: "UART / 4-bit SD Selector & Debug"
- note removed: "UART0_RX"
- note removed: "UART0_TX"
- moved on the sheet: D1, D2, D3, H1, H2, H3, H4, R1, R13, R14, R15, R18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
